File: prod_board/prod_board.sch (EAGLE design)
At the start: 31 parts

Commit message: prod board layout v1
Parts:
- SERVO: value SPDTSWITCH -> (none); device fab:SPDTSWITCH -> pinhead:PINHD-1X3
Connections:
- net GND: now also SERVO.1; no longer SERVO.3
- net N$14: now also SERVO.3; no longer SERVO.1
Changed lines of the file:
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@@
 <part name="P+1" library="supply1" library_urn="urn:adsk.eagle:library:371" deviceset="+5V" device=""/>
 <part name="GND1" library="supply1" library_urn="urn:adsk.eagle:library:371" deviceset="GND" device=""/>
-<part name="SERVO" library="fab" deviceset="SPDTSWITCH" device=""/>
 <part name="U$2" library="fab" deviceset="LED" device="FAB1206"/>
 <part name="U$3" library="fab" deviceset="LED" device="FAB1206"/>
@@
 <part name="GND3" library="supply1" library_urn="urn:adsk.eagle:library:371" deviceset="GND" device=""/>
 <part name="P+2" library="supply1" library_urn="urn:adsk.eagle:library:371" deviceset="+5V" device=""/>
+<part name="SERVO" library="pinhead" library_urn="urn:adsk.eagle:library:325" deviceset="PINHD-1X3" device="" package3d_urn="urn:adsk.eagle:package:22458/2"/>
 </parts>
 <sheets>
@@
 <instance part="P+1" gate="1" x="81.28" y="104.14"/>
 <instance part="GND1" gate="1" x="81.28" y="33.02"/>
-<instance part="SERVO" gate="G$1" x="93.98" y="17.78"/>
 <instance part="U$2" gate="G$1" x="162.56" y="63.5"/>
 <instance part="U$3" gate="G$1" x="167.64" y="66.04" rot="R180"/>
@@
 <instance part="GND3" gate="1" x="106.68" y="12.7" rot="R90"/>
 <instance part="P+2" gate="1" x="106.68" y="17.78" rot="R270"/>
+<instance part="SERVO" gate="A" x="78.74" y="17.78" rot="R180"/>
 </instances>
 <busses>
@@
 </segment>
 <segment>
-<pinref part="SERVO" gate="G$1" pin="2"/>
 <pinref part="P+2" gate="1" pin="+5V"/>
-<wire x1="93.98" y1="17.78" x2="104.14" y2="17.78" width="0.1524" layer="91"/>
+<pinref part="SERVO" gate="A" pin="2"/>
+<wire x1="104.14" y1="17.78" x2="81.28" y2="17.78" width="0.1524" layer="91"/>
 </segment>
 </net>
@@
 </segment>
 <segment>
-<pinref part="SERVO" gate="G$1" pin="3"/>
 <pinref part="GND3" gate="1" pin="GND"/>
-<wire x1="93.98" y1="12.7" x2="104.14" y2="12.7" width="0.1524" layer="91"/>
+<wire x1="88.9" y1="12.7" x2="104.14" y2="12.7" width="0.1524" layer="91"/>
+<wire x1="88.9" y1="12.7" x2="88.9" y2="15.24" width="0.1524" layer="91"/>
+<pinref part="SERVO" gate="A" pin="1"/>
+<wire x1="88.9" y1="15.24" x2="81.28" y2="15.24" width="0.1524" layer="91"/>
 </segment>
 </net>
@@
 <wire x1="124.46" y1="45.72" x2="104.14" y2="45.72" width="0.1524" layer="91"/>
 <wire x1="104.14" y1="45.72" x2="104.14" y2="22.86" width="0.1524" layer="91"/>
-<pinref part="SERVO" gate="G$1" pin="1"/>
-<wire x1="104.14" y1="22.86" x2="93.98" y2="22.86" width="0.1524" layer="91"/>
+<wire x1="104.14" y1="22.86" x2="88.9" y2="22.86" width="0.1524" layer="91"/>
+<wire x1="88.9" y1="22.86" x2="88.9" y2="20.32" width="0.1524" layer="91"/>
+<pinref part="SERVO" gate="A" pin="3"/>
+<wire x1="88.9" y1="20.32" x2="81.28" y2="20.32" width="0.1524" layer="91"/>
 </segment>
 </net>
@@
 will not be understood (or retained) with this version.
 </note>
+<note version="8.3" severity="warning">
+Since Version 8.3, EAGLE supports the association of 3D packages
+with devices in libraries, schematics, and board files. Those 3D
+packages will not be understood (or retained) with this version.
+</note>
 </compatibility>

Commit message: main board into production v1
Parts:
- removed U$18, U$19, U$20, U$21: LEDFAB1206, fab:LEDFAB1206
Connections:
- removed net N$9: R9.2, U$15.A, U$16.C, U$17.A, U$18.C, U$19.A, U$20.C, U$21.A, U$6.C
- new net N$15: R9.2, U$15.A, U$16.C, U$17.A, U$6.C
- net N$5: no longer U$20.A, U$21.C
- net N$6: no longer U$18.A, U$19.C
Other:
- moved on the sheet: U$22
Changed lines of the file:
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@@
 <part name="U$16" library="fab" deviceset="LED" device="FAB1206"/>
 <part name="U$17" library="fab" deviceset="LED" device="FAB1206"/>
-<part name="U$18" library="fab" deviceset="LED" device="FAB1206"/>
-<part name="U$19" library="fab" deviceset="LED" device="FAB1206"/>
-<part name="U$20" library="fab" deviceset="LED" device="FAB1206"/>
-<part name="U$21" library="fab" deviceset="LED" device="FAB1206"/>
 <part name="U$22" library="solidlib" deviceset="ARDUINO_CONN" device=""/>
 <part name="GND4" library="supply1" library_urn="urn:adsk.eagle:library:371" deviceset="GND" device=""/>
@@
 <instance part="U$16" gate="G$1" x="228.6" y="38.1"/>
 <instance part="U$17" gate="G$1" x="233.68" y="40.64" rot="R180"/>
-<instance part="U$18" gate="G$1" x="241.3" y="50.8"/>
-<instance part="U$19" gate="G$1" x="246.38" y="53.34" rot="R180"/>
-<instance part="U$20" gate="G$1" x="254" y="63.5"/>
-<instance part="U$21" gate="G$1" x="259.08" y="66.04" rot="R180"/>
 <instance part="U$22" gate="G$1" x="124.46" y="60.96"/>
 <instance part="GND4" gate="1" x="104.14" y="68.58" rot="R270"/>
@@
 <junction x="162.56" y="68.58"/>
 <pinref part="R5" gate="G$1" pin="2"/>
-<pinref part="U$20" gate="G$1" pin="A"/>
-<wire x1="220.98" y1="68.58" x2="254" y2="68.58" width="0.1524" layer="91"/>
-<junction x="220.98" y="68.58"/>
-<pinref part="U$21" gate="G$1" pin="C"/>
-<wire x1="254" y1="68.58" x2="259.08" y2="68.58" width="0.1524" layer="91"/>
-<junction x="254" y="68.58"/>
 </segment>
 </net>
@@
 <junction x="167.64" y="55.88"/>
 <pinref part="R6" gate="G$1" pin="2"/>
-<pinref part="U$18" gate="G$1" pin="A"/>
-<wire x1="208.28" y1="55.88" x2="241.3" y2="55.88" width="0.1524" layer="91"/>
-<junction x="208.28" y="55.88"/>
-<pinref part="U$19" gate="G$1" pin="C"/>
-<wire x1="241.3" y1="55.88" x2="246.38" y2="55.88" width="0.1524" layer="91"/>
-<junction x="241.3" y="55.88"/>
 </segment>
 </net>
@@
 </segment>
 </net>
-<net name="N$9" class="0">
-<segment>
-<pinref part="R9" gate="G$1" pin="2"/>
-<wire x1="154.94" y1="17.78" x2="193.04" y2="17.78" width="0.1524" layer="91"/>
-<pinref part="U$6" gate="G$1" pin="C"/>
-<wire x1="193.04" y1="17.78" x2="198.12" y2="17.78" width="0.1524" layer="91"/>
-<wire x1="198.12" y1="17.78" x2="228.6" y2="17.78" width="0.1524" layer="91"/>
-<wire x1="228.6" y1="17.78" x2="233.68" y2="17.78" width="0.1524" layer="91"/>
-<wire x1="233.68" y1="17.78" x2="241.3" y2="17.78" width="0.1524" layer="91"/>
-<wire x1="241.3" y1="17.78" x2="246.38" y2="17.78" width="0.1524" layer="91"/>
-<wire x1="246.38" y1="17.78" x2="254" y2="17.78" width="0.1524" layer="91"/>
-<wire x1="254" y1="17.78" x2="259.08" y2="17.78" width="0.1524" layer="91"/>
-<wire x1="193.04" y1="22.86" x2="193.04" y2="17.78" width="0.1524" layer="91"/>
-<junction x="193.04" y="17.78"/>
-<pinref part="U$15" gate="G$1" pin="A"/>
-<wire x1="198.12" y1="22.86" x2="198.12" y2="17.78" width="0.1524" layer="91"/>
-<junction x="198.12" y="17.78"/>
-<pinref part="U$21" gate="G$1" pin="A"/>
-<wire x1="259.08" y1="17.78" x2="259.08" y2="60.96" width="0.1524" layer="91"/>
-<pinref part="U$20" gate="G$1" pin="C"/>
-<wire x1="254" y1="60.96" x2="254" y2="17.78" width="0.1524" layer="91"/>
-<junction x="254" y="17.78"/>
-<pinref part="U$17" gate="G$1" pin="A"/>
-<wire x1="233.68" y1="35.56" x2="233.68" y2="17.78" width="0.1524" layer="91"/>
-<junction x="233.68" y="17.78"/>
-<pinref part="U$16" gate="G$1" pin="C"/>
-<wire x1="228.6" y1="35.56" x2="228.6" y2="17.78" width="0.1524" layer="91"/>
-<junction x="228.6" y="17.78"/>
-<pinref part="U$18" gate="G$1" pin="C"/>
-<wire x1="241.3" y1="48.26" x2="241.3" y2="17.78" width="0.1524" layer="91"/>
-<junction x="241.3" y="17.78"/>
-<pinref part="U$19" gate="G$1" pin="A"/>
-<wire x1="246.38" y1="48.26" x2="246.38" y2="17.78" width="0.1524" layer="91"/>
-<junction x="246.38" y="17.78"/>
-</segment>
-</net>
 <net name="N$3" class="0">
 <segment>
@@
 </segment>
 </net>
+<net name="N$15" class="0">
+<segment>
+<pinref part="U$17" gate="G$1" pin="A"/>
+<wire x1="233.68" y1="35.56" x2="233.68" y2="17.78" width="0.1524" layer="91"/>
+<pinref part="R9" gate="G$1" pin="2"/>
+<wire x1="154.94" y1="17.78" x2="193.04" y2="17.78" width="0.1524" layer="91"/>
+<pinref part="U$6" gate="G$1" pin="C"/>
+<wire x1="193.04" y1="22.86" x2="193.04" y2="17.78" width="0.1524" layer="91"/>
+<junction x="193.04" y="17.78"/>
+<wire x1="193.04" y1="17.78" x2="198.12" y2="17.78" width="0.1524" layer="91"/>
+<pinref part="U$15" gate="G$1" pin="A"/>
+<wire x1="198.12" y1="22.86" x2="198.12" y2="17.78" width="0.1524" layer="91"/>
+<junction x="198.12" y="17.78"/>
+<wire x1="198.12" y1="17.78" x2="228.6" y2="17.78" width="0.1524" layer="91"/>
+<wire x1="228.6" y1="17.78" x2="233.68" y2="17.78" width="0.1524" layer="91"/>
+<junction x="228.6" y="17.78"/>
+<pinref part="U$16" gate="G$1" pin="C"/>
+<wire x1="228.6" y1="35.56" x2="228.6" y2="17.78" width="0.1524" layer="91"/>
+</segment>
+</net>
